File: STM32F401/STM32F401.kicad_pcb (KiCad board)
At the start: 4 copper layers, 26.6 x 19.8 mm, 57 parts, among them U1 STM32F401CCUx, U2 MCP73832-2-OT, U3 MCP1811A-033TT, Y1 Crystal_GND24_Small, Y2 Crystal_Small

Commit message: Swap `PA13` with `PA11`
Use `PA11` as the `CHG_STAT` pin to free up `PA13` which is needed for
SWD.
Connections:
- H12 pad 1: PA11 -> PA13
- U1 pad 32: PA11 -> CHG_STAT
- U1 pad 34: CHG_STAT -> PA13
Routing:
- net PA11: track 9.53 -> 0.00 mm, vias 1 -> 0
- net PA13: track 0.00 -> 8.87 mm, vias 0 -> 1
- net CHG_STAT: track 3.65 -> 2.97 mm, vias 2 -> 0
